Commit message: [FT] loading the urdf in drake
Changed "package://" paths to absolute paths. This is a hack, needs to
be changed back. Made all the fricton parameters of the joints to be 0.
This was not the case in the original urdf description

File: core/nextagea_description/urdf/NextageaOpenObj.urdf (robot description, URDF)
Before this commit: robot NextageAOpen, 18 links, 17 joints
Links:
- link CHEST_JOINT0_Link: geometry collision box size=0.085 0.5 0.0365; collision box size=0.17 0.29 0.225
- link HEAD_JOINT0_Link: geometry collision cylinder length=0.135 radius=0.035; visual mesh filename=/home/aditya/Documents/projects/avro22/ARO_Practical_2022/s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
- link HEAD_JOINT1_Link: geometry collision box size=0.27 0.22 0.115; visual mesh filename=/home/aditya/Documents/projects/avro22/ARO_Practical_2022/s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
- link LARM_JOINT0_Link: geometry collision box size=0.048 0.1 0.035; collision box size=0.1 0.0815 0.19
- link LARM_JOINT1_Link: geometry collision box size=0.08 0.11 0.28; collision box size=0.122 0.0338 0.062
- link LARM_JOINT2_Link: geometry collision box size=0.119 0.125 0.1; collision cylinder length=0.04 radius=0.047
- link LARM_JOINT3_Link: geometry collision box size=0.093 0.112 0.037; collision cylinder length=0.12 radius=0.035
- link LARM_JOINT4_Link: geometry collision box size=0.04 0.118 0.06; collision cylinder length=0.08 radius=0.037
- link LARM_JOINT5_Link: geometry collision box size=0.057 0.106 0.042; collision cylinder length=0.07 radius=0.037
- link RARM_JOINT0_Link: geometry collision box size=0.048 0.1 0.035; collision box size=0.1 0.0815 0.19
- link RARM_JOINT1_Link: geometry collision box size=0.08 0.11 0.28; collision box size=0.122 0.0338 0.062
- link RARM_JOINT2_Link: geometry collision box size=0.119 0.125 0.1; collision cylinder length=0.04 radius=0.047
- link RARM_JOINT3_Link: geometry collision box size=0.093 0.112 0.037; collision cylinder length=0.12 radius=0.035
- link RARM_JOINT4_Link: geometry collision box size=0.04 0.118 0.06; collision cylinder length=0.08 radius=0.037
- link RARM_JOINT5_Link: geometry collision box size=0.057 0.106 0.042; collision cylinder length=0.07 radius=0.037
- link WAIST: geometry collision cylinder length=0.376 radius=0.06; visual mesh filename=/home/aditya/Documents/projects/avro22/ARO_Practical_2022/s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
- link nextage_base: geometry collision box size=0.585 0.585 0.72; collision sphere radius=0.03

Commit message: [WIP] inverse dynamics added to nextage manipulation station

File: core/nextagea_description/urdf/NextageaOpenObj.urdf (robot description, URDF)
Before this commit: robot NextageAOpen, 18 links, 17 joints
Links:
- link CHEST_JOINT0_Link: geometry collision box size=0.085 0.5 0.0365; collision box size=0.17 0.29 0.225
- link HEAD_JOINT0_Link: geometry collision cylinder length=0.135 radius=0.035; visual mesh filename=package://nextagea_description/urdf/meshes/HEAD_JOINT0_Link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
- link HEAD_JOINT1_Link: geometry collision box size=0.27 0.22 0.115; visual mesh filename=package://nextagea_description/urdf/meshes/HEAD_JOINT1_Link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
- link LARM_JOINT0_Link: geometry collision box size=0.048 0.1 0.035; collision box size=0.1 0.0815 0.19
- link LARM_JOINT1_Link: geometry collision box size=0.08 0.11 0.28; collision box size=0.122 0.0338 0.062
- link LARM_JOINT2_Link: geometry collision box size=0.119 0.125 0.1; collision cylinder length=0.04 radius=0.047
- link LARM_JOINT3_Link: geometry collision box size=0.093 0.112 0.037; collision cylinder length=0.12 radius=0.035
- link LARM_JOINT4_Link: geometry collision box size=0.04 0.118 0.06; collision cylinder length=0.08 radius=0.037
- link LARM_JOINT5_Link: geometry collision box size=0.057 0.106 0.042; collision cylinder length=0.07 radius=0.037
- link RARM_JOINT0_Link: geometry collision box size=0.048 0.1 0.035; collision box size=0.1 0.0815 0.19
- link RARM_JOINT1_Link: geometry collision box size=0.08 0.11 0.28; collision box size=0.122 0.0338 0.062
- link RARM_JOINT2_Link: geometry collision box size=0.119 0.125 0.1; collision cylinder length=0.04 radius=0.047
- link RARM_JOINT3_Link: geometry collision box size=0.093 0.112 0.037; collision cylinder length=0.12 radius=0.035
- link RARM_JOINT4_Link: geometry collision box size=0.04 0.118 0.06; collision cylinder length=0.08 radius=0.037
- link RARM_JOINT5_Link: geometry collision box size=0.057 0.106 0.042; collision cylinder length=0.07 radius=0.037
- link WAIST: geometry collision cylinder length=0.376 radius=0.06; visual mesh filename=package://nextagea_description/urdf/meshes/WAIST_Link_mesh.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
- link nextage_base: geometry collision box size=0.585 0.585 0.72; collision sphere radius=0.03
